File: Hardware/KiCad/6x-BPF-FRONTEND.kicad_pcb (KiCad board)
At the start: 2 copper layers, 177.3 x 64.9 mm, 88 parts, among them K1 G6K-2, K2 G6K-2, K3 G6K-2, K4 G6K-2, K5 G6K-2, K6 G6K-2, K7 G6K-2, Q1 BC547, U1 ULN2003, U2 4028, U3 LM1117T-3.3, U4 LM7805_TO220

Commit message: Correzione bug
Corretto alcuni valori che nello schema erano errati
Parts:
- C12, C15: value 180uF -> 180pF
- C2: value 10uF -> 10nF
Changed lines of the file:
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@@
 			)
 		)
-		(property "Value" "10uF"
+		(property "Value" "10nF"
 			(at -5.6682 -0.27 0)
 			(layer "F.Fab")
@@
 		)
 		(fp_text user "${REFERENCE}"
-			(at 2.54 -4.27 0)
+			(at -3.9236 -2.55 0)
 			(layer "F.Fab")
 			(effects
@@
 			)
 		)
-		(property "Value" "180uF"
+		(property "Value" "180pF"
 			(at -5.746 -0.17 0)
 			(layer "F.Fab")
@@
 			)
 		)
-		(property "Value" "180uF"
+		(property "Value" "180pF"
 			(at -5.746 -0.17 0)
 			(layer "F.Fab")
@@
 		)
 		(fp_text user "${REFERENCE}"
-			(at 2.54 -4.27 0)
+			(at -4.1986 -2.7 0)
 			(layer "F.Fab")
 			(effects
