File: Hardware/KiCad/6x-BPF-FRONTEND.kicad_sch (KiCad schematic)
At the start: 87 parts, among them J1 RF OUT, J2 RF IN, J3 +12V, J4 Band, J5 Att., J6 PBF VFO, K1 G6K-2, K2 G6K-2, K3 G6K-2, K4 G6K-2, K5 G6K-2, K6 G6K-2, K7 G6K-2, Q1 BC547, U1 ULN2003, U2 4028, U3 LM1117T-3.3, U4 LM7805_TO220

Commit message: Correzione bug
Corretto alcuni valori che nello schema erano errati
Parts:
- C12, C15: value 180uF -> 180pF
- C2: value 10uF -> 10nF
Changed lines of the file:
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@@
 		(dnp no)
 		(property "Reference" "C13"
-			(at 211.836 52.07 0)
+			(at 210.82 52.07 0)
 			(effects
 				(font
@@
 			)
 		)
-		(property "Value" "180uF"
+		(property "Value" "180pF"
 			(at 234.442 47.752 90)
 			(effects
@@
 			)
 		)
-		(property "Value" "180uF"
+		(property "Value" "180pF"
 			(at 234.442 59.436 90)
 			(effects
@@
 			)
 		)
-		(property "Value" "10uF"
+		(property "Value" "10nF"
 			(at 117.094 54.61 0)
 			(effects

Commit message: Aggiornato distinta materiali
Parts:
- C1: value 12.2nF -> 10+2.2 nF
- C4: value 1.22nF -> 1nF+220pF
Changed lines of the file:
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@@
 			)
 		)
-		(property "Value" "12.2nF"
+		(property "Value" "10+2.2 nF"
 			(at 146.05 56.388 90)
 			(effects
@@
 			)
 		)
-		(property "Value" "1.22nF"
+		(property "Value" "1nF+220pF"
 			(at 144.78 103.378 90)
 			(effects
